File: AdderRev1.sch (EAGLE design)
At the start: 20 parts, among them IC1 4008N

Commit message: Added design frame and title block to sch file and added images to repository and readme
Other:
- note added: "1"
- moved on the sheet: IC1, IC1P, INPUTA, INPUTB, LED1, LED2, LED3, LED4, POWERJACK, R1, R10, R11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
